Commit message: Fetch without collision for anything but the base

File: robots/fetch_armless.urdf (robot description, URDF)
Before this commit: robot fetch, 7 links, 6 joints
Links:
- link head_pan_link: geometry visual mesh filename=package://fetch_description/meshes/head_pan_link.dae
- link head_tilt_link: geometry visual mesh filename=package://fetch_description/meshes/head_tilt_link.dae
- link torso_fixed_link: geometry visual mesh filename=package://fetch_description/meshes/torso_fixed_link.dae
- link torso_lift_link: geometry visual mesh filename=package://fetch_description/meshes/torso_lift_link.dae

Commit message: Replaced the robot's collision geometry

File: robots/fetch_armless.urdf (robot description, URDF)
Before this commit: robot fetch, 7 links, 6 joints
Links:
- link base_collision_link: geometry collision cylinder length=1.5 radius=0.3; visual mesh filename=package://fetch_description/meshes/base_link.dae
